File: power-systems-v3.kicad_pcb (KiCad board)
At the start: 4 copper layers, 94 x 30 mm, 52 parts, among them J1 Conn_01x02_Socket, J10 Conn_01x03_Pin, J2 Conn_01x02_Socket, J3 Conn_01x08_Pin, J4 Conn_01x08_Pin, J5 Conn_01x08_Pin, J6 Conn_01x02_Socket, J7 Conn_01x02_Socket, J9 Conn_01x03_Pin, Q1 Q_PMOS, SW1 SW_SPST, U1 INA226, U2 LMR51430YDDCR, U3 LMR51430YDDCR, U6 AL8843SP-13, U7 AL8843SP-13

Commit message: final pcb
Parts:
- added REF**: MountingHole_2.7mm_M2.5, MountingHole:MountingHole_2.7mm_M2.5, F.Cu at (220.0, 42.0)
- added REF**: MountingHole_2.7mm_M2.5, MountingHole:MountingHole_2.7mm_M2.5, F.Cu at (133.5, 42.0)
- added REF**: MountingHole_2.7mm_M2.5, MountingHole:MountingHole_2.7mm_M2.5, F.Cu at (133.5, 79.0)
- added REF**: MountingHole_2.7mm_M2.5, MountingHole:MountingHole_2.7mm_M2.5, F.Cu at (220.0, 79.0)
Routing:
- net 12V: track 104.2 -> 138.3 mm, vias 4 -> 44
- net 5out: track 56.7 -> 35.7 mm
- net Net-(U2-SW): track 12.4 -> 22.4 mm
- net Net-(D11-A): track 28.0 -> 36.2 mm, vias 2 -> 6
- net Net-(D12-A): vias 2 -> 6
- net GND: vias 16 -> 18
- added copper zone on F.Cu, net /LED1+
- added copper zone on F.Cu, net /LED1-
- added copper zone on F.Cu, net /LED2+
- added copper zone on F.Cu, net /LED2-
- added copper zone on B.Cu, net 12V
- added copper zone on F.Cu, net Net-(U2-SW)
- added copper zone on F.Cu, net Net-(U3-CB)
- added copper zone on F.Cu, net Net-(U3-SW)
Other:
- board size 94 x 30 mm -> 95 x 44 mm
